Commit message: 4/27 gazebo custom world, total launch

File: mini_pupper_ros/mini_pupper_description/urdf/mini_pupper_description.urdf.xacro (robot description, xacro)
@@ -102,5 +102,5 @@
   </joint>
   <link
-    name="lidar">
+    name="lidar_link">
     <inertial>
       <origin
@@ -149,18 +149,4 @@
     <parent
       link="base_link" />
-    <child
-      link="lidar" />
-    <axis
-      xyz="0 0 0" />
-  </joint>
-  <link name="lidar_link" />
-  <joint
-    name="lidar_link_joint"
-    type="fixed">
-    <origin
-      xyz="0 0 0"
-      rpy="0 0 0" />
-    <parent
-      link="lidar" />
     <child
       link="lidar_link" />
@@ -1740,9 +1726,8 @@
     <material>Gazebo/FlatBlack</material>
   </gazebo>
-  <gazebo reference="lidar">
+  <gazebo reference="lidar_link">
     <material>Gazebo/FlatBlack</material>
     <sensor type="ray" name="lidar">
       <always_on>true</always_on>
-      <visualize>false</visualize>
       <update_rate>30</update_rate>
       <pose>0 0 0 0 0 0</pose>
@@ -1773,5 +1758,5 @@
         </ros>
         <output_type>sensor_msgs/LaserScan</output_type>
-        <frame_name>lidar</frame_name>
+        <frame_name>lidar_link</frame_name>
         <!--min_intensity>100.0</min_intensity-->
       </plugin>
@@ -1796,17 +1781,4 @@
     </plugin>
   </gazebo>
-  <gazebo>
-    <plugin filename="libhector_gazebo_ros_imu.so" name="imu_controller">
-      <updateRate>50.0</updateRate>
-      <bodyName>imu_link</bodyName>
-      <topicName>imu/data</topicName>
-      <accelDrift>0.005 0.005 0.005</accelDrift>
-      <accelGaussianNoise>0.005 0.005 0.005</accelGaussianNoise>
-      <rateDrift>0.005 0.005 0.005 </rateDrift>
-      <rateGaussianNoise>0.005 0.005 0.005 </rateGaussianNoise>
-      <headingDrift>0.005</headingDrift>
-      <headingGaussianNoise>0.005</headingGaussianNoise>
-    </plugin>
-  </gazebo>
   <link name="imu_link">
     <inertial>
@@ -1820,4 +1792,16 @@
     <child link="imu_link"/>
   </joint>
+  <gazebo reference="imu_link">
+    <sensor name="imu_controller" type="imu">
+      <always_on>true</always_on>
+      <update_rate>50</update_rate>
+      <plugin name="gazebo_ros_imu_sensor" filename="libgazebo_ros_imu_sensor.so">
+          <ros>
+              <namespace>/imu</namespace>
+              <argument>~/out:=data</argument>
+          </ros>
+      </plugin>
+    </sensor>
+  </gazebo>
   <!--xacro:sensor_d435 parent="base_link">
   <origin xyz="0.08 0.0 0.07" rpy="0 0 0" />
